Commit message: upgrade the obstacle_avoidance algorithm

File: 3rd_mid_GazeboSimulation/mid_project/urdf/robot.xacro (robot description, xacro)
@@ -9,5 +9,5 @@
         <inertial>
             <mass value="${chassis_mass}" />
-            <origin xyz="0 0 0.3" rpy="0 0 0" />
+            <origin xyz="0 0 0.2" rpy="0 0 0" />
             <inertia ixx="1.5417" ixy="0" ixz="0" iyy="3.467" iyz="0" izz="4.742" />
         </inertial>
